Commit message: Update

File: description/robot.urdf.xacro (robot description, xacro)
@@ -2,3 +2,5 @@
 <robot xmlns:xacro="http://www.ros.org/wiki/xacro"  name="robot">
     <xacro:include filename="robot_core.xacro"/>
+    <xacro:include filename="gazebo_control.xacro"/>
+    <xacro:include filename="lidar.xacro"/>
 </robot>

File: description/robot_core.xacro (robot description, xacro)
@@ -14,4 +14,7 @@
         <color rgba="0 0 0 1"/>
     </material>
+    <material name="red" >
+        <color rgba="1 0 0 1"/>
+    </material>
     <!-- BASE LINK  -->
     <link name="base_link">
@@ -21,115 +24,105 @@
         <parent link ="base_link"/>
         <child link ="chassis"/>
-        <origin xyz="-0.05 0 0"/>
+        <origin xyz="-0.1 0 0"/>
     </joint>
     <link name="chassis">
         <visual>
-            <origin xyz="0.07 0 0.02"/>
+            <origin xyz="0.15 0 0.075" rpy="0 0 0"/>
             <geometry>
-                <box size="0.20 0.16 0.05"/>
+                <box size="0.3 0.3 0.15"/>
             </geometry>
             <material name="white"/>
         </visual>
         <collision>
-            <origin xyz="0.07 0 0.02"/>
+            <origin xyz="0.15 0 0.075" rpy="0 0 0"/>
             <geometry>
-                <box size="0.20 0.16 0.05"/>
+                <box size="0.3 0.3 0.15"/>
             </geometry>
         </collision>
-        <xacro:inertial_box mass="1" x="0.20" y="0.16" z="0.05">
-            <origin xyz="0.07 0 0.02" rpy="0 0 0"/>
+        <xacro:inertial_box mass="0.5" x="0.3" y="0.3" z="0.15">
+            <origin xyz="0.15 0 0.075" rpy="0 0 0"/>
         </xacro:inertial_box>
     </link>
-    <!-- LEFT WHEEL 1 -->
-    <joint name="left_wheel_joint_1" type="continuous">
+    <gazebo reference="chassis">
+        <material>Gazebo/White</material>
+    </gazebo>
+    <!-- LEFT WHEEL -->
+    <joint name="left_wheel_joint" type="continuous">
         <parent link="base_link"/>
-        <child link="left_wheel_1"/>
-        <origin xyz="-0.06 0.08 0" rpy="-${pi/2} 0 0"/>
+        <child link="left_wheel"/>
+        <origin xyz="0 0.175 0" rpy="-${pi/2} 0 0"/>
         <axis xyz="0 0 1"/>
     </joint>
-    <link name="left_wheel_1">
+    <link name="left_wheel">
         <visual>
-            <material name="black"/>
             <geometry>
-                <cylinder radius="0.035" length="0.04"/>
+                <cylinder length="0.04" radius="0.05" />
             </geometry>
+            <material name="blue"/>
         </visual>
         <collision>
             <geometry>
-                <cylinder radius="0.035" length="0.04"/>
+                <cylinder length="0.04" radius="0.05" />
             </geometry>
         </collision>
-        <xacro:inertial_cylinder mass="0.2" length="0.04" radius="0.035">
+        <xacro:inertial_cylinder mass="0.1" length="0.05" radius="0.05">
             <origin xyz="0 0 0" rpy="0 0 0"/>
         </xacro:inertial_cylinder>
     </link>
-<!-- LEFT WHEEL 2 -->
-    <joint name="left_wheel_joint_2" type="continuous">
+    <gazebo reference="left_wheel">
+        <material>Gazebo/Blue</material>
+    </gazebo>
+<!-- RIGHT WHEEL -->
+    <joint name="right_wheel_joint" type="continuous">
         <parent link="base_link"/>
-        <child link="left_wheel_2"/>
-        <origin xyz="0.09 0.08 0" rpy="-${pi/2} 0 0"/>
-        <axis xyz="0 0 1"/>
+        <child link="right_wheel"/>
+        <origin xyz="0 -0.175 0" rpy="${pi/2} 0 0"/>
+        <axis xyz="0 0 -1"/>
     </joint>
-    <link name="left_wheel_2">
+    <link name="right_wheel">
         <visual>
-            <material name="black"/>
             <geometry>
-                <cylinder radius="0.035" length="0.04"/>
+                <cylinder length="0.04" radius="0.05" />
             </geometry>
+            <material name="blue"/>
         </visual>
         <collision>
             <geometry>
-                <cylinder radius="0.035" length="0.04"/>
+                <cylinder length="0.04" radius="0.05" />
             </geometry>
         </collision>
-        <xacro:inertial_cylinder mass="0.2" length="0.04" radius="0.035">
+        <xacro:inertial_cylinder mass="0.1" length="0.05" radius="0.05">
             <origin xyz="0 0 0" rpy="0 0 0"/>
         </xacro:inertial_cylinder>
     </link>
-<!-- RIGHT WHEEL 1 -->
-    <joint name="right_wheel_joint_1" type="continuous">
-        <parent link="base_link"/>
-        <child link="right_wheel_1"/>
-        <origin xyz="-0.06 -0.08 0" rpy="${pi/2} 0 0"/>
-        <axis xyz="0 0 1"/>
+    <gazebo reference="right_wheel">
+        <material>Gazebo/Blue</material>
+    </gazebo>
+    <!-- Caster Wheel -->
+    <joint name="caster_wheel_joint" type='fixed'>
+        <parent link="chassis"/>
+        <child link="caster_wheel"/>
+        <origin xyz="0.24 0 0"/>
     </joint>
-    <link name="right_wheel_1">
+    <link name="caster_wheel">
         <visual>
+            <geometry>
+                <sphere radius="0.05"/>
+            </geometry>
             <material name="black"/>
-            <geometry>
-                <cylinder radius="0.035" length="0.04"/>
-            </geometry>
         </visual>
         <collision>
             <geometry>
-                <cylinder radius="0.035" length="0.04"/>
+                <sphere radius="0.05"/>
             </geometry>
         </collision>
-        <xacro:inertial_cylinder mass="0.2" length="0.04" radius="0.035">
+        <xacro:inertial_sphere mass="0.1" radius="0.05">
             <origin xyz="0 0 0" rpy="0 0 0"/>
-        </xacro:inertial_cylinder>
+        </xacro:inertial_sphere>
     </link>
-    <!-- RIGHT WHEEL 2 -->
-    <joint name="right_wheel_joint_2" type="continuous">
-        <parent link="base_link"/>
-        <child link="right_wheel_2"/>
-        <origin xyz="0.09 -0.08 0" rpy="${pi/2} 0 0"/>
-        <axis xyz="0 0 1"/>
-    </joint>
-    <link name="right_wheel_2">
-        <visual>
-            <material name="black"/>
-            <geometry>
-                <cylinder radius="0.035" length="0.04"/>
-            </geometry>
-        </visual>
-        <collision>
-            <geometry>
-                <cylinder radius="0.035" length="0.04"/>
-            </geometry>
-        </collision>
-        <xacro:inertial_cylinder mass="0.2" length="0.04" radius="0.035">
-            <origin xyz="0 0 0" rpy="0 0 0"/>
-        </xacro:inertial_cylinder>
-    </link>
+    <gazebo reference="caster_wheel">
+        <material>Gazebo/Black</material>
+        <mu1 value="0.001"/>
+        <mu2 value="0.001"/>
+    </gazebo>
     </robot>
